File: Electronics/power_management.kicad_sch (KiCad schematic)
At the start: 0 parts

Commit message: basic power supply layout some minor design notes. charge ic likely to change. possibly bridge out fuel gague
Parts:
- added BT1: 18650, Battery:BatteryHolder_Keystone_1042_1x18650, symbol Device:Battery_Cell
- added C4: 1u, Capacitor_SMD:C_0603_1608Metric_Pad1.08x0.95mm_HandSolder, symbol Device:C
- added C5, C6: 10u, Capacitor_SMD:C_0603_1608Metric_Pad1.08x0.95mm_HandSolder, symbol Device:C
- added J2: USB_C_Receptacle_USB2.0_14P, symbol Connector:USB_C_Receptacle_USB2.0_14P
- added R1: 100m, Resistor_SMD:R_1210_3225Metric_Pad1.30x2.65mm_HandSolder, symbol Device:R
- added R4: 2k, Resistor_SMD:R_0402_1005Metric_Pad0.72x0.64mm_HandSolder, symbol Device:R
- added R5, R6: 5.1k, Resistor_SMD:R_0402_1005Metric_Pad0.72x0.64mm_HandSolder, symbol Device:R
- added R7: 1M, Resistor_SMD:R_0402_1005Metric_Pad0.72x0.64mm_HandSolder, symbol Device:R
- added SW43: SW_DPDT_x2, symbol Switch:SW_DPDT_x2
- added U3: TLV75733PDBV, Package_TO_SOT_SMD:SOT-23-5, symbol Regulator_Linear:TLV75733PDBV
- added U4: LTC2942, Package_DFN_QFN:DFN-6-1EP_3x2mm_P0.5mm_EP1.65x1.35mm, symbol Battery_Management:LTC2942
- added U5: MCP73812T-435I-OT, Package_TO_SOT_SMD:SOT-23-5, symbol Battery_Management:MCP73812T-435I-OT
Connections:
- new net: J2.S1 (SHIELD), R7.1
- new net: BT1.1 (+), R1.2, U4.6 (SENSE-)
- new net: J2.B5 (CC2), R5.1
- new net: C4.1, R1.1, SW43.2 (B), U4.1 (SENSE+), U5.3 (V_{BAT})
- new net: SW43.3 (C), U3.1 (IN), U3.3 (EN)
- new net: R4.1, U5.5 (PROG)
- new net: J2.A4 (VBUS), J2.A9 (VBUS), J2.B4 (VBUS), J2.B9 (VBUS), U5.1 (CE), U5.4 (V_{DD})
- new net: J2.A5 (CC1), R6.1
- new net +3V3: C5.1, C6.1, U3.5 (OUT)
- new net 0: BT1.2 (-), C4.2, C5.2, C6.2, J2.A1 (GND), J2.A12 (GND), J2.B1 (GND), J2.B12 (GND), R4.2, R5.2, R6.2, R7.2, U3.2 (GND), U4.2 (GND), U5.2 (V_{SS})
- new net BATTERY_SCL: U4.3 (SCL)
- new net BATTERY_SDA: U4.4 (SDA)
- new net USB_DM: J2.A7 (D-), J2.B7 (D-)
- new net USB_DP: J2.A6 (D+), J2.B6 (D+)
- no-connect marks 0 -> 1
